Commit message: fix abduction direction

File: pupper_controller/src/pupperv2/data/pupper_no_mesh.urdf (robot description, URDF)
Before this commit: robot pupper_v2_dji, 17 links, 16 joints
Joints:
- joint leftFrontLegMotor: axis 0 -1.0 0 -> 0 1.0 0
- joint rightRearLegMotor: axis 0 1.0 0 -> 0 -1.0 0

Commit message: Fix abduction angles. Add configurable friction. Update package reqs.

File: pupper_controller/src/pupperv2/data/pupper_no_mesh.urdf (robot description, URDF)
Before this commit: robot pupper_v2_dji, 17 links, 16 joints
Joints:
- removed joint leftFrontLegMotor
- removed joint leftRearLegMotor
- removed joint rightFrontLegMotor
- removed joint rightRearLegMotor
- added joint leftFrontAbductionMotor: type revolute, parent pupper_v2_dji_chassis, child leftFrontLeg, origin xyz=0.047 -0.1015 0 rpy=0 0 0, axis 0 -1.0 0, limit lower=-0.7854 upper=0.7854 effort=0 velocity=0
- added joint leftRearAbductionMotor: type revolute, parent pupper_v2_dji_chassis, child leftRearLeg, origin xyz=0.047 0.0985 0 rpy=0 0 0, axis 0 -1.0 0, limit lower=-0.7854 upper=0.7854 effort=0 velocity=0
- added joint rightFrontAbductionMotor: type revolute, parent pupper_v2_dji_chassis, child rightFrontLeg, origin xyz=-0.047 -0.103 0 rpy=0 0 -3.14159, axis 0 1.0 0, limit lower=-0.7854 upper=0.7854 effort=0 velocity=0
- added joint rightRearAbductionMotor: type revolute, parent pupper_v2_dji_chassis, child rightRearLeg, origin xyz=-0.047 0.097 0 rpy=0 0 -3.14159, axis 0 1.0 0, limit lower=-0.7854 upper=0.7854 effort=0 velocity=0
