Commit message: Bug fixing for the is_sim and is_physical arguments to ensure PCs not running the physical model can run the code without physical library errors. Changing of config parameters to match Dingo V2 (Current physical implementation of the robot). Quick check of angles shows them not working correctly, needs further investigation

File: dingo_ws/src/dingo_description/urdf/notspot.urdf (robot description, URDF)
Before this commit: robot notspot, 17 links, 16 joints
Links:
- link FL1: geometry visual mesh filename=package://dingo_description/meshes/FL1_obj.obj
- link FL2: geometry collision cylinder length=0.125 radius=0.014; visual mesh filename=package://dingo_description/meshes/L2_obj.obj
- link FL3: geometry collision cylinder length=0.06 radius=0.007; visual mesh filename=package://dingo_description/meshes/L3_obj.obj
- link FR1: geometry visual mesh filename=package://dingo_description/meshes/FR1_obj.obj
- link FR2: geometry collision cylinder length=0.125 radius=0.014; visual mesh filename=package://dingo_description/meshes/R2_obj.obj
- link FR3: geometry collision cylinder length=0.06 radius=0.007; visual mesh filename=package://dingo_description/meshes/R3_obj.obj
- link RL1: geometry visual mesh filename=package://dingo_description/meshes/RL1_obj.obj
- link RL2: geometry collision cylinder length=0.125 radius=0.014; visual mesh filename=package://dingo_description/meshes/L2_obj.obj
- link RL3: geometry collision cylinder length=0.06 radius=0.007; visual mesh filename=package://dingo_description/meshes/L3_obj.obj
- link RR1: geometry visual mesh filename=package://dingo_description/meshes/RR1_obj.obj
- link RR2: geometry collision cylinder length=0.125 radius=0.014; visual mesh filename=package://dingo_description/meshes/R2_obj.obj
- link RR3: geometry collision cylinder length=0.06 radius=0.007; visual mesh filename=package://dingo_description/meshes/R3_obj.obj
- link base_link: geometry collision box size=0.25 0.1285 0.055; visual mesh filename=package://dingo_description/meshes/body_obj.obj
