Commit message: Added publishing of joint space and task space goals to the code, including custom messages to nicely define them in topics and an Angle message for angles. Deleted old values in config and moved length definitions there, and updated them for the current robot shape. Further fixes on URDF file to make it more stable

File: dingo_ws/src/dingo_description/urdf/dingo copy.urdf (robot description, URDF)
Before this commit: robot dingo, 17 links, 16 joints
Links:
- link FL_link1: mass 0.30000000 -> 0.2
- link FL_link2: mass 0.10000000 -> 0.05
- link FL_link3: mass 0.10000000 -> 0.05
- link FL_link4: mass 0.02000000 -> 0.01
- link FR_link1: mass 0.30000000 -> 0.2
- link FR_link2: mass 0.10000000 -> 0.05
- link FR_link3: mass 0.10000000 -> 0.05
- link FR_link4: mass 0.02000000 -> 0.01
- link RL_link1: mass 0.30000000 -> 0.2
- link RL_link2: mass 0.10000000 -> 0.05
- link RL_link3: mass 0.10000000 -> 0.05
- link RL_link4: mass 0.02000000 -> 0.01
- link RR_link1: mass 0.30000000 -> 0.2
- link RR_link2: mass 0.10000000 -> 0.05
- link RR_link3: mass 0.10000000 -> 0.05
- link RR_link4: mass 0.02000000 -> 0.01
- link base_link: mass 2.50000000 -> 2.2
Joints:
- joint FL_theta1: limit lower=-0.785398 upper=0.785398 effort=${effort_limit} velocity=3 -> (none)
- joint FL_theta2: limit lower=-3 upper=3 effort=${effort_limit} velocity=3 -> (none)
- joint FL_theta3: limit lower=-3 upper=3 effort=${effort_limit} velocity=3 -> (none)
- joint FR_theta1: limit lower=-0.785398 upper=0.785398 effort=${effort_limit} velocity=3 -> (none)
- joint FR_theta2: limit lower=-3 upper=3 effort=${effort_limit} velocity=3 -> (none)
- joint FR_theta3: limit lower=-3 upper=3 effort=${effort_limit} velocity=3 -> (none)
- joint RL_theta1: limit lower=-0.785398 upper=0.785398 effort=${effort_limit} velocity=3 -> (none)
- joint RL_theta2: limit lower=-3 upper=3 effort=${effort_limit} velocity=3 -> (none)
- joint RL_theta3: limit lower=-3 upper=3 effort=${effort_limit} velocity=3 -> (none)
- joint RR_theta1: limit lower=-0.785398 upper=0.785398 effort=${effort_limit} velocity=3 -> (none)
- joint RR_theta2: limit lower=-3 upper=3 effort=${effort_limit} velocity=3 -> (none)
- joint RR_theta3: limit lower=-3 upper=3 effort=${effort_limit} velocity=3 -> (none)
