Commit message: Various changes to urdf, kinematics and the addition of a battery checking script via digital

File: dingo_ws/src/dingo_description/urdf/dingo.urdf (robot description, URDF)
Before this commit: robot dingo, 17 links, 16 joints
Joints:
- joint FL_theta1: type continuous -> revolute
- joint FL_theta2: type continuous -> revolute
- joint FL_theta3: type continuous -> revolute
- joint FR_theta1: type continuous -> revolute
- joint FR_theta2: type continuous -> revolute
- joint FR_theta3: type continuous -> revolute
- joint RL_theta1: type continuous -> revolute
- joint RL_theta2: type continuous -> revolute
- joint RL_theta3: type continuous -> revolute
- joint RR_theta1: type continuous -> revolute
- joint RR_theta2: type continuous -> revolute
- joint RR_theta3: type continuous -> revolute

Commit message: Changes to kinematics and sim to fix some issues, including walking backwards

File: dingo_ws/src/dingo_description/urdf/dingo.urdf (robot description, URDF)
Before this commit: robot dingo, 17 links, 16 joints
Links:
- link base_link: mass 2.50000000 -> 0.81776
